Commit message: testing

File: tripteron.urdf (robot description, URDF)
Before this commit: robot tripteron, 3 links, 2 joints
Links:
- link base_1: geometry visual cylinder length=0.5 radius=0.1
- link base_link: geometry visual box size=0.5 0.5 0.5
Joints:
- joint dist1: limit lower=0 upper=20.0 effort=1000.0 velocity=0.5 -> (none); origin xyz=-0.4 0 0.3 rpy=0 0 0 -> xyz=0.5 0.25 0.5  rpy=0 0 0; type prismatic -> continuous

Commit message: Base Model URDF Done

File: tripteron.urdf (robot description, URDF)
Before this commit: robot tripteron, 3 links, 2 joints
Links:
- removed link base_1
- removed link base_link
- added link base_link_BL
- added link base_link_BR
- added link base_link_FL
- added link base_link_FR
- added link leftArm_1
- added link leftArm_2
- added link leftArm_3
- added link leftArm_4
- added link rightArm_1
- added link rightArm_2
- added link rightArm_3
- added link rightArm_4
Joints:
- removed joint dist1
- removed joint rSlider
- added joint base_link_BR: type continuous, parent base_link_BR, child base_link_BL, origin xyz=0 0.2 0 rpy=0 0 0, axis 1 0 0
- added joint start_joint_BR: type continuous, parent world, child base_link_BR, origin xyz=1.2 0 0 rpy=0 0 0, axis 1 0 0
- added joint start_joint_FL: type continuous, parent base_link_FR, child base_link_FL, origin xyz=0 0.2 0 rpy=0 0 0, axis 1 0 0
- added joint start_joint_FR: type continuous, parent world, child base_link_FR, origin xyz=0.2 0 0 rpy=0 0 0, axis 1 0 0
- added joint theta1: type continuous, parent base_link_FR, child rightArm_1, origin xyz=0.2 -0.2 0.2  rpy=0 0 0, axis 1 0 0
- added joint theta2: type continuous, parent rightArm_1, child rightArm_2, origin xyz=0.2 0.2 0.2  rpy=0 0 0, axis 1 0 0
- added joint theta3: type continuous, parent base_link_FL, child leftArm_1, origin xyz=0.2 0.2 0.2  rpy=0 0 0, axis 1 0 0
- added joint theta4: type continuous, parent leftArm_1, child leftArm_2, origin xyz=0.2 -0.2 0.2  rpy=0 0 0, axis 1 0 0
- added joint theta5: type continuous, parent base_link_BR, child rightArm_3, origin xyz=-0.2 -0.2 0.2  rpy=0 0 0, axis 1 0 0
- added joint theta6: type continuous, parent rightArm_3, child rightArm_4, origin xyz=-0.2 0.2 0.2  rpy=0 0 0, axis 1 0 0
- added joint theta7: type continuous, parent base_link_BL, child leftArm_3, origin xyz=-0.2 0.2 0.2  rpy=0 0 0, axis 1 0 0
- added joint theta8: type continuous, parent leftArm_3, child leftArm_4, origin xyz=-0.2 -0.2 0.2  rpy=0 0 0, axis 1 0 0
