Commit message: added ROS and Tripteron body

File: URDF/tripteronBody.urdf (robot description, URDF)
Before this commit: robot tripteronBody, 0 links, 0 joints
Links:
- added link base_link; visual box size=0.1524 0.1524 0.1016
- added link lowerArm_four; visual cylinder length=0.1524 radius=0.0127
- added link lowerArm_one; visual cylinder length=0.1524 radius=0.0127
- added link lowerArm_three; visual cylinder length=0.1524 radius=0.0127
- added link lowerArm_two; visual cylinder length=0.1524 radius=0.0127
- added link railAttach_four; visual box size=0.00001016 0.000001016 0.0001016
- added link railAttach_one; visual box size=0.1016 0.1016 0.1016
- added link railAttach_three; visual box size=0.00001016 0.000001016 0.0001016
- added link railAttach_two; visual box size=0.1016 0.1016 0.1016
- added link upperArm_four; visual cylinder length=0.1524 radius=0.0127
- added link upperArm_one; visual cylinder length=0.1524 radius=0.0127
- added link upperArm_three; visual cylinder length=0.1524 radius=0.0127
- added link upperArm_two; visual cylinder length=0.1524 radius=0.0127
Joints:
- added joint theta1: type continuous, parent base_link, child upperArm_one, origin xyz=0.0500 -0.0500 -0.0508 rpy=-0.7854 -0.7854 0, axis 1 0 0
- added joint theta10: type continuous, parent base_link, child upperArm_four, origin xyz=-0.0500 0.0500 -0.0508 rpy=2.3562 0 -2.3562, axis 1 0 0
- added joint theta11: type continuous, parent upperArm_four, child lowerArm_four, origin xyz=0 0 0.1524 rpy=0 1.0472 0, axis 1 0 0
- added joint theta12: type continuous, parent lowerArm_four, child railAttach_four, origin xyz=0 0 0.1524 rpy=0.7854 -1.5708 0 , axis 1 0 0
- added joint theta2: type continuous, parent upperArm_one, child lowerArm_one, origin xyz=0 0 -0.1524 rpy=-1.5708 0 0, axis 1 0 0
- added joint theta3: type continuous, parent lowerArm_one, child railAttach_one, origin xyz=0 0 0.1524 rpy=-0.7854 -0.7854 -1.5708, axis 0 1 0
- added joint theta4: type continuous, parent base_link, child upperArm_two, origin xyz=0.0500 0.0500 -0.0508 rpy=3.9269 -0.7854 0, axis 1 0 0
- added joint theta5: type continuous, parent upperArm_two, child lowerArm_two, origin xyz=0 0 0.1524 rpy=-1.5708 0 0, axis 1 0 0
- added joint theta6: type continuous, parent lowerArm_two, child railAttach_two, origin xyz=0 0 0.1524 rpy=-0.7854 0.7854 -1.5708 , axis 0 1 0
- added joint theta7: type continuous, parent base_link, child upperArm_three, origin xyz=-0.0500 -0.0500 -0.0508 rpy=2.3562 0 -0.7854, axis 1 0 0
- added joint theta8: type continuous, parent upperArm_three, child lowerArm_three, origin xyz=0 0 0.1524 rpy=0 -1.0472 0, axis 1 0 0
- added joint theta9: type continuous, parent lowerArm_three, child railAttach_three, origin xyz=0 0 0.1524 rpy=0 0 0, axis 1 0 0

Commit message: fixed mistake on urdf

File: URDF/tripteronBody.urdf (robot description, URDF)
Before this commit: robot tripteronBody, 13 links, 12 joints
Joints:
- joint theta1: axis 1 0 0 -> 0 0 1
