Commit message: adjusted resting position

File: Description/tripteronBody.xacro (robot description, xacro)
@@ -1,4 +1,4 @@
 <?xml version="1.0"?>
-<robot xmlns:xacro="http://www.ros.org/wiki/xacro" name="tripteronBody">
+<robot xmlns:xacro="http://www.ros.org/wiki/xacro" name="tripteron">
 <!-- *************************************************** -->
 <!-- ******************** Kinematics ******************* -->
@@ -20,12 +20,12 @@
           <parent link="base_link"/>
           <child  link="upperArm_one"/>
-          <origin xyz="${O_x} -${O_y} -${O_z}" rpy="-${pi/4} -${pi/4} 0"/>
-          <axis   xyz="0 0 1"/>
+          <origin xyz="${O_x} -${O_y} -${O_z}" rpy="-${pi/2} -${pi/4} 0"/>
+          <axis   xyz="1 0 0"/>
      </joint>
      <link name="upperArm_one">
           <visual>
-               <origin xyz="0 0 -${limbLng/2}" rpy="0 0 0"/>
+               <origin xyz="0 0 -${toplimbLng/2}" rpy="0 0 0"/>
                <geometry>
-                    <cylinder radius="${limbRad}" length="${limbLng}"/>
+                    <cylinder radius="${limbRad}" length="${toplimbLng}"/>
                </geometry>
                <material name="cyan"/>
@@ -36,12 +36,12 @@
           <parent link="upperArm_one"/>
           <child  link="lowerArm_one"/>
-          <origin xyz="0 0 -${limbLng}" rpy="-${pi/2} 0 0"/>
+          <origin xyz="0 0 -${toplimbLng}" rpy="-${pi/4} 0 0"/>
           <axis   xyz="1 0 0"/>
      </joint>
      <link name="lowerArm_one">
           <visual>
-               <origin xyz="0 0 ${limbLng/2}" rpy="0 0 0"/>
+               <origin xyz="0 0 ${bottomlimbLng/2}" rpy="0 0 0"/>
                <geometry>
-                    <cylinder radius="${limbRad}" length="${limbLng}"/>
+                    <cylinder radius="${limbRad}" length="${bottomlimbLng}"/>
                </geometry>
                <material name="green"/>
@@ -52,5 +52,5 @@
           <parent link="lowerArm_one"/>
           <child  link="railAttach_one"/>
-          <origin xyz="0 0 ${limbLng}" rpy="0 0 0"/>
+          <origin xyz="0 0 ${bottomlimbLng}" rpy="-${pi/4} -${pi/4} -${pi/2}"/>
           <axis   xyz="0 1 0"/>
      </joint>
@@ -61,12 +61,12 @@
           <parent link="base_link"/>
           <child  link="upperArm_two"/>
-          <origin xyz="${O_x} ${O_y} -${O_z}" rpy="${5*pi/4} -${pi/4} 0"/>
+          <origin xyz="${O_x} ${O_y} -${O_z}" rpy="-${pi/2} -${pi/4} 0"/>
           <axis   xyz="1 0 0"/>
      </joint>
      <link name="upperArm_two">
           <visual>
-               <origin xyz="0 0 0.0762" rpy="0 0 0"/>
+               <origin xyz="0 0 ${toplimbLng/2}" rpy="0 0 0"/>
                <geometry>
-                    <cylinder radius="${limbRad}" length="${limbLng}"/>
+                    <cylinder radius="${limbRad}" length="${toplimbLng}"/>
                </geometry>
                <material name="cyan"/>
@@ -77,12 +77,12 @@
           <parent link="upperArm_two"/>
           <child  link="lowerArm_two"/>
-          <origin xyz="0 0 ${limbLng}" rpy="-${pi/2} 0 0"/>
+          <origin xyz="0 0 ${toplimbLng}" rpy="-${3*pi/4} 0 0"/>
           <axis   xyz="1 0 0"/>
      </joint>
      <link name="lowerArm_two">
           <visual>
-               <origin xyz="0 0 ${limbLng/2}" rpy="0 0 0"/>
+               <origin xyz="0 0 ${bottomlimbLng/2}" rpy="0 0 0"/>
                <geometry>
-                    <cylinder radius="${limbRad}" length="${limbLng}"/>
+                    <cylinder radius="${limbRad}" length="${bottomlimbLng}"/>
                </geometry>
                <material name="green"/>
@@ -93,5 +93,5 @@
           <parent link="lowerArm_two"/>
           <child  link="railAttach_two"/>
-          <origin xyz="0 0 ${limbLng}" rpy="0 0 0"/>
+          <origin xyz="0 0 ${bottomlimbLng}" rpy="-${pi/4} ${pi/4} -${pi/2}"/>
           <axis   xyz="0 1 0"/>
      </joint>
@@ -102,12 +102,12 @@
           <parent link="base_link"/>
           <child  link="upperArm_three"/>
-          <origin xyz="-${O_x} -${O_y} -${O_z}" rpy="${3*pi/4} 0 -${pi/4}"/>  <!-- Come back later to mess with the yaw  -0.7854 -->
+          <origin xyz="-${O_x} -${O_y} -${O_z}" rpy="${pi/3} ${pi/4} -${pi/4}"/>  <!-- Come back later to mess with the yaw  -${pi/4} -->
           <axis   xyz="1 0 0"/>
      </joint>
      <link name="upperArm_three">
           <visual>
-               <origin xyz="0 0 ${limbLng/2}" rpy="0 0 0"/>
+               <origin xyz="0 0 ${toplimbLng/2}" rpy="0 0 0"/>
                <geometry>
-                    <cylinder radius="${limbRad}" length="${limbLng}"/>
+                    <cylinder radius="${limbRad}" length="${toplimbLng}"/>
                </geometry>
                <material name="cyan"/>
@@ -118,12 +118,12 @@
           <parent link="upperArm_three"/>
           <child  link="lowerArm_three"/>
-          <origin xyz="0 0 ${limbLng}" rpy="0 -${pi/3} 0"/>
+          <origin xyz="0 0 ${toplimbLng}" rpy="-${2*pi/3} 0 ${pi}"/>
           <axis   xyz="1 0 0"/>
      </joint>
      <link name="lowerArm_three">
           <visual>
-               <origin xyz="0 0 ${limbLng/2}" rpy="0 0 0"/>
+               <origin xyz="0 0 ${bottomlimbLng/2}" rpy="0 0 0"/>
                <geometry>
-                    <cylinder radius="${limbRad}" length="${limbLng}"/>
+                    <cylinder radius="${limbRad}" length="${bottomlimbLng}"/>
                </geometry>
                <material name="green"/>
@@ -134,5 +134,5 @@
           <parent link="lowerArm_three"/>
           <child  link="railAttach_three"/>
-          <origin xyz="0 0 ${limbLng}" rpy="0 0 0"/>
+          <origin xyz="0 0 ${bottomlimbLng}" rpy="-${pi/4} ${pi/4} 0"/>
           <axis   xyz="1 0 0"/>
      </joint>
@@ -143,12 +143,12 @@
           <parent link="base_link"/>
           <child  link="upperArm_four"/>
-          <origin xyz="-${O_x} ${O_y} -${O_z}" rpy="${3*pi/4} 0 -${3*pi/4}"/>  <!-- Come back later to mess with the yaw  -0.7854 -->
+          <origin xyz="-${O_x} ${O_y} -${O_z}" rpy="-${pi/3} ${pi/4} ${pi/4}"/>  <!-- Come back later to mess with the yaw  -0.7854 -->
           <axis   xyz="1 0 0"/>
      </joint>
      <link name="upperArm_four">
           <visual>
-               <origin xyz="0 0 ${limbLng/2}" rpy="0 0 0"/>
+               <origin xyz="0 0 ${toplimbLng/2}" rpy="0 0 0"/>
                <geometry>
-                    <cylinder radius="${limbRad}" length="${limbLng}"/>
+                    <cylinder radius="${limbRad}" length="${toplimbLng}"/>
                </geometry>
                <material name="cyan"/>
@@ -159,12 +159,12 @@
           <parent link="upperArm_four"/>
           <child  link="lowerArm_four"/>
-          <origin xyz="0 0 ${limbLng}" rpy="0 ${pi/3} 0"/>  <!-- 1.0472  | 0.7854 -->
+          <origin xyz="0 0 ${toplimbLng}" rpy="${2*pi/3} 0 ${pi}"/>
           <axis   xyz="1 0 0"/>
      </joint>
      <link name="lowerArm_four">
           <visual>
-               <origin xyz="0 0 ${limbLng/2}" rpy="0 0 0"/>
+               <origin xyz="0 0 ${bottomlimbLng/2}" rpy="0 0 0"/>
                <geometry>
-                    <cylinder radius="${limbRad}" length="${limbLng}"/>
+                    <cylinder radius="${limbRad}" length="${bottomlimbLng}"/>
                </geometry>
                <material name="green"/>
@@ -175,5 +175,5 @@
           <parent link="lowerArm_four"/>
           <child  link="railAttach_four"/>
-          <origin xyz="0 0 ${limbLng}" rpy="0 0 0 "/>  <!-- 1.0472  2.3562 -1.5708  |0.7854 -1.5708 0-->
+          <origin xyz="0 0 ${bottomlimbLng}" rpy="-${pi/4} ${pi/4} 0"/>  <!-- rpy="${pi/3} ${3*pi/4} -${pi/2}"  |${pi/4} -${pi/2} 0-->
           <axis   xyz="1 0 0"/>
      </joint>

File: Description/tripteronBodyFull.xacro (robot description, xacro)
@@ -20,12 +20,12 @@
           <parent link="base_link"/>
           <child  link="upperArm_one"/>
-          <origin xyz="${O_x} -${O_y} -${O_z}" rpy="-${pi/4} -${pi/4} 0"/>
-          <axis   xyz="0 0 1"/>
+          <origin xyz="${O_x} -${O_y} -${O_z}" rpy="-${pi/2} -${pi/4} 0"/>
+          <axis   xyz="1 0 0"/>
      </joint>
      <link name="upperArm_one">
           <visual>
-               <origin xyz="0 0 -${limbLng/2}" rpy="0 0 0"/>
-               <geometry>
-                    <cylinder radius="${limbRad}" length="${limbLng}"/>
+               <origin xyz="0 0 -${toplimbLng/2}" rpy="0 0 0"/>
+               <geometry>
+                    <cylinder radius="${limbRad}" length="${toplimbLng}"/>
                </geometry>
                <material name="cyan"/>
@@ -36,12 +36,12 @@
           <parent link="upperArm_one"/>
           <child  link="lowerArm_one"/>
-          <origin xyz="0 0 -${limbLng}" rpy="-${pi/2} 0 0"/>
+          <origin xyz="0 0 -${toplimbLng}" rpy="-${pi/4} 0 0"/>
           <axis   xyz="1 0 0"/>
      </joint>
      <link name="lowerArm_one">
           <visual>
-               <origin xyz="0 0 ${limbLng/2}" rpy="0 0 0"/>
-               <geometry>
-                    <cylinder radius="${limbRad}" length="${limbLng}"/>
+               <origin xyz="0 0 ${bottomlimbLng/2}" rpy="0 0 0"/>
+               <geometry>
+                    <cylinder radius="${limbRad}" length="${bottomlimbLng}"/>
                </geometry>
                <material name="green"/>
@@ -52,5 +52,5 @@
           <parent link="lowerArm_one"/>
           <child  link="railAttach_one"/>
-          <origin xyz="0 0 ${limbLng}" rpy="-${pi/4} -${pi/4} -${pi/2}"/>
+          <origin xyz="0 0 ${bottomlimbLng}" rpy="-${pi/4} -${pi/4} -${pi/2}"/>
           <axis   xyz="0 1 0"/>
      </joint>
@@ -69,12 +69,12 @@
           <parent link="base_link"/>
           <child  link="upperArm_two"/>
-          <origin xyz="${O_x} ${O_y} -${O_z}" rpy="${5*pi/4} -${pi/4} 0"/>
+          <origin xyz="${O_x} ${O_y} -${O_z}" rpy="-${pi/2} -${pi/4} 0"/>
           <axis   xyz="1 0 0"/>
      </joint>
      <link name="upperArm_two">
           <visual>
-               <origin xyz="0 0 0.0762" rpy="0 0 0"/>
-               <geometry>
-                    <cylinder radius="${limbRad}" length="${limbLng}"/>
+               <origin xyz="0 0 ${toplimbLng/2}" rpy="0 0 0"/>
+               <geometry>
+                    <cylinder radius="${limbRad}" length="${toplimbLng}"/>
                </geometry>
                <material name="cyan"/>
@@ -85,12 +85,12 @@
           <parent link="upperArm_two"/>
           <child  link="lowerArm_two"/>
-          <origin xyz="0 0 ${limbLng}" rpy="-${pi/2} 0 0"/>
+          <origin xyz="0 0 ${toplimbLng}" rpy="-${3*pi/4} 0 0"/>
           <axis   xyz="1 0 0"/>
      </joint>
      <link name="lowerArm_two">
           <visual>
-               <origin xyz="0 0 ${limbLng/2}" rpy="0 0 0"/>
-               <geometry>
-                    <cylinder radius="${limbRad}" length="${limbLng}"/>
+               <origin xyz="0 0 ${bottomlimbLng/2}" rpy="0 0 0"/>
+               <geometry>
+                    <cylinder radius="${limbRad}" length="${bottomlimbLng}"/>
                </geometry>
                <material name="green"/>
@@ -101,5 +101,5 @@
           <parent link="lowerArm_two"/>
           <child  link="railAttach_two"/>
-          <origin xyz="0 0 ${limbLng}" rpy="-${pi/4} ${pi/4} -${pi/2}"/>
+          <origin xyz="0 0 ${bottomlimbLng}" rpy="-${pi/4} ${pi/4} -${pi/2}"/>
           <axis   xyz="0 1 0"/>
      </joint>
@@ -118,12 +118,12 @@
           <parent link="base_link"/>
           <child  link="upperArm_three"/>
-          <origin xyz="-${O_x} -${O_y} -${O_z}" rpy="${3*pi/4} 0 -${pi/4}"/>  <!-- Come back later to mess with the yaw  -0.7854 -->
+          <origin xyz="-${O_x} -${O_y} -${O_z}" rpy="${pi/3} ${pi/4} -${pi/4}"/>  <!-- Come back later to mess with the yaw  -${pi/4} -->
           <axis   xyz="1 0 0"/>
      </joint>
      <link name="upperArm_three">
           <visual>
-               <origin xyz="0 0 ${limbLng/2}" rpy="0 0 0"/>
-               <geometry>
-                    <cylinder radius="${limbRad}" length="${limbLng}"/>
+               <origin xyz="0 0 ${toplimbLng/2}" rpy="0 0 0"/>
+               <geometry>
+                    <cylinder radius="${limbRad}" length="${toplimbLng}"/>
                </geometry>
                <material name="cyan"/>
@@ -134,12 +134,12 @@
           <parent link="upperArm_three"/>
           <child  link="lowerArm_three"/>
-          <origin xyz="0 0 ${limbLng}" rpy="0 -${pi/3} 0"/>
+          <origin xyz="0 0 ${toplimbLng}" rpy="-${2*pi/3} 0 ${pi}"/>
           <axis   xyz="1 0 0"/>
      </joint>
      <link name="lowerArm_three">
           <visual>
-               <origin xyz="0 0 ${limbLng/2}" rpy="0 0 0"/>
-               <geometry>
-                    <cylinder radius="${limbRad}" length="${limbLng}"/>
+               <origin xyz="0 0 ${bottomlimbLng/2}" rpy="0 0 0"/>
+               <geometry>
+                    <cylinder radius="${limbRad}" length="${bottomlimbLng}"/>
                </geometry>
                <material name="green"/>
@@ -150,12 +150,12 @@
           <parent link="lowerArm_three"/>
           <child  link="railAttach_three"/>
-          <origin xyz="0 0 ${limbLng}" rpy="0 0 0"/>
+          <origin xyz="0 0 ${bottomlimbLng}" rpy="-${pi/4} ${pi/4} 0"/>
           <axis   xyz="1 0 0"/>
      </joint>
      <link name="railAttach_three">
           <visual>
-               <origin xyz="0 -${slider_size/2} 0" rpy="0 0 0"/>
-               <geometry>
-                    <xacro:Cube size="0.000001"/>
+               <origin xyz="-${slider_size/2} 0 0" rpy="0 0 0"/>
+               <geometry>
+                    <xacro:Cube size="${slider_size}"/>
                </geometry>
                <material name="red"/>
@@ -167,12 +167,12 @@
           <parent link="base_link"/>
           <child  link="upperArm_four"/>
-          <origin xyz="-${O_x} ${O_y} -${O_z}" rpy="${3*pi/4} 0 -${3*pi/4}"/>  <!-- Come back later to mess with the yaw  -0.7854 -->
+          <origin xyz="-${O_x} ${O_y} -${O_z}" rpy="-${pi/3} ${pi/4} ${pi/4}"/>  <!-- Come back later to mess with the yaw  -0.7854 -->
           <axis   xyz="1 0 0"/>
      </joint>
      <link name="upperArm_four">
           <visual>
-               <origin xyz="0 0 ${limbLng/2}" rpy="0 0 0"/>
-               <geometry>
-                    <cylinder radius="${limbRad}" length="${limbLng}"/>
+               <origin xyz="0 0 ${toplimbLng/2}" rpy="0 0 0"/>
+               <geometry>
+                    <cylinder radius="${limbRad}" length="${toplimbLng}"/>
                </geometry>
                <material name="cyan"/>
@@ -183,12 +183,12 @@
           <parent link="upperArm_four"/>
           <child  link="lowerArm_four"/>
-          <origin xyz="0 0 ${limbLng}" rpy="0 ${pi/3} 0"/>
+          <origin xyz="0 0 ${toplimbLng}" rpy="${2*pi/3} 0 ${pi}"/>
           <axis   xyz="1 0 0"/>
      </joint>
      <link name="lowerArm_four">
           <visual>
-               <origin xyz="0 0 ${limbLng/2}" rpy="0 0 0"/>
-               <geometry>
-                    <cylinder radius="${limbRad}" length="${limbLng}"/>
+               <origin xyz="0 0 ${bottomlimbLng/2}" rpy="0 0 0"/>
+               <geometry>
+                    <cylinder radius="${limbRad}" length="${bottomlimbLng}"/>
                </geometry>
                <material name="green"/>
@@ -199,10 +199,10 @@
           <parent link="lowerArm_four"/>
           <child  link="railAttach_four"/>
-          <origin xyz="0 0 ${limbLng}" rpy="-${pi/10} 0 -${pi/4}"/>  <!-- rpy="${pi/3} ${3*pi/4} -${pi/2}"  |${pi/4} -${pi/2} 0-->
+          <origin xyz="0 0 ${bottomlimbLng}" rpy="-${pi/4} ${pi/4} 0"/>  <!-- rpy="${pi/3} ${3*pi/4} -${pi/2}"  |${pi/4} -${pi/2} 0-->
           <axis   xyz="1 0 0"/>
      </joint>
      <link name="railAttach_four">
           <visual>
-               <origin xyz="0 -${slider_size/2} 0" rpy="0 0 0"/>
+               <origin xyz="-${slider_size/2} 0 0" rpy="0 0 0"/>
                <geometry>
                     <xacro:Cube size="${slider_size}"/>

File: Description/util.xacro (robot description, xacro)
@@ -1,4 +1,4 @@
 <?xml version="1.0"?>
-<robot xmlns:xacro="http://www.ros.org/wiki/xacro">
+<robot xmlns:xacro="http://www.ros.org/wiki/xacro" name="tripteron">
     <!-- Util class-->
     <!--                         numbers:                    -->
@@ -6,5 +6,6 @@
     <!-- 0.0254 = 1in    --> <!-- 0.0127 = 0.5in -->
     <xacro:property name="limbRad" value="0.0127" />
-    <xacro:property name="limbLng" value="0.1524" />
+    <xacro:property name="toplimbLng" value="0.1524" />
+    <xacro:property name="bottomlimbLng" value="0.2155" /> <!-- 0.2155  -->
     <xacro:property name="pltf_l" value="0.1524" />
     <xacro:property name="pltf_w" value="0.1524" />
