Commit message: integrated xacro with ros

File: urdf/tripteronBody.urdf.xacro (robot description, xacro)
@@ -5,4 +5,10 @@
 <!-- *************************************************** -->
 <xacro:include filename="util.xacro"/>
+    <link name="world"/>
+     <joint name="base_joint" type="fixed">
+        <origin xyz="1.5 1.0 0.25" rpy="0 0 0"/>
+        <parent link="world"/>
+        <child link="base_link"/>
+    </joint>
 <!-- URDF relations to IRL are in meters-->
      <link name="base_link">
@@ -55,13 +61,5 @@
           <axis   xyz="0 1 0"/>
      </joint>
-     <link name="railAttach_one">
-          <visual>
-               <origin xyz="0 -${slider_size/2} 0" rpy="0 0 0"/>
-               <geometry>
-                    <xacro:Cube size="${slider_size}"/>
-               </geometry>
-               <material name="red"/>
-          </visual>
-     </link>
+     <link name="railAttach_one"/>
 <!-- ******************** ARM TWO ******************* -->
      <!-- Base_link to Upper arm  -->
@@ -104,13 +102,5 @@
           <axis   xyz="0 1 0"/>
      </joint>
-     <link name="railAttach_two">
-          <visual>
-               <origin xyz="0 -${slider_size/2} 0" rpy="0 0 0"/>
-               <geometry>
-                    <xacro:Cube size="${slider_size}"/>
-               </geometry>
-               <material name="red"/>
-          </visual>
-     </link>
+     <link name="railAttach_two"/>
 <!-- ******************** ARM THREE ******************* -->
      <!-- Base_link to Upper arm  -->
@@ -153,13 +143,5 @@
           <axis   xyz="1 0 0"/>
      </joint>
-     <link name="railAttach_three">
-          <visual>
-               <origin xyz="-${slider_size/2} 0 0" rpy="0 0 0"/>
-               <geometry>
-                    <xacro:Cube size="${slider_size}"/>
-               </geometry>
-               <material name="red"/>
-          </visual>
-     </link>
+     <link name="railAttach_three"/>
 <!-- ******************** ARM FOUR ******************* -->
      <!-- Base_link to Upper arm  -->
@@ -202,12 +184,4 @@
           <axis   xyz="1 0 0"/>
      </joint>
-     <link name="railAttach_four">
-          <visual>
-               <origin xyz="-${slider_size/2} 0 0" rpy="0 0 0"/>
-               <geometry>
-                    <xacro:Cube size="${slider_size}"/>
-               </geometry>
-               <material name="red"/>
-          </visual>
-     </link>
+     <link name="railAttach_four"/>
  </robot>

File: urdf/tripteronBodyFull.urdf.xacro (robot description, xacro)
@@ -5,4 +5,10 @@
 <!-- *************************************************** -->
 <xacro:include filename="util.xacro"/>
+    <link name="world"/>
+    <joint name="base_joint" type="fixed">
+        <origin xyz="1.5 1.0 0.25" rpy="0 0 0"/>
+        <parent link="world"/>
+        <child link="base_link"/>
+    </joint>
 <!-- URDF relations to IRL are in meters-->
      <link name="base_link">
@@ -49,11 +55,20 @@
      </link>
      <!-- Lower Arm to rail attachment -->
-     <joint name="theta3" type="continuous">
+     <joint name="theta3" type="prismatic">
           <parent link="lowerArm_one"/>
           <child  link="railAttach_one"/>
           <origin xyz="0 0 ${bottomlimbLng}" rpy="-${pi/4} -${pi/4} -${pi/2}"/>
-          <axis   xyz="0 1 0"/>
-     </joint>
-     <link name="railAttach_one"/>
+          <axis   xyz="0 0 1"/>
+          <limit lower="${lLim_front}" upper="${uLim_front}" velocity="100" effort="100"/>
+     </joint>
+     <link name="railAttach_one">
+          <visual>
+               <origin xyz="0 -${slider_size/2} 0" rpy="0 0 0"/>
+               <geometry>
+                    <xacro:Cube size="${slider_size}"/>
+               </geometry>
+               <material name="red"/>
+          </visual>
+     </link>
 <!-- ******************** ARM TWO ******************* -->
      <!-- Base_link to Upper arm  -->
@@ -90,11 +105,20 @@
      </link>
      <!-- Lower Arm to rail attachment -->
-     <joint name="theta6" type="continuous">
+     <joint name="theta6" type="prismatic">
           <parent link="lowerArm_two"/>
           <child  link="railAttach_two"/>
           <origin xyz="0 0 ${bottomlimbLng}" rpy="-${pi/4} ${pi/4} -${pi/2}"/>
-          <axis   xyz="0 1 0"/>
-     </joint>
-     <link name="railAttach_two"/>
+          <axis   xyz="0 0 1"/>
+          <limit lower="${lLim_front}" upper="${uLim_front}" velocity="100" effort="100"/>
+     </joint>
+     <link name="railAttach_two">
+          <visual>
+               <origin xyz="0 -${slider_size/2} 0" rpy="0 0 0"/>
+               <geometry>
+                    <xacro:Cube size="${slider_size}"/>
+               </geometry>
+               <material name="red"/>
+          </visual>
+     </link>
 <!-- ******************** ARM THREE ******************* -->
      <!-- Base_link to Upper arm  -->
@@ -131,11 +155,20 @@
      </link>
      <!-- Lower Arm to rail attachment -->
-     <joint name="theta9" type="continuous">
+     <joint name="theta9" type="prismatic">
           <parent link="lowerArm_three"/>
           <child  link="railAttach_three"/>
           <origin xyz="0 0 ${bottomlimbLng}" rpy="-${pi/4} ${pi/4} 0"/>
-          <axis   xyz="1 0 0"/>
-     </joint>
-     <link name="railAttach_three"/>
+          <axis   xyz="0 1 0"/>
+          <limit lower="${lLim_back}" upper="${uLim_back}" velocity="100" effort="100"/>
+     </joint>
+     <link name="railAttach_three">
+          <visual>
+               <origin xyz="-${slider_size/2} 0 0" rpy="0 0 0"/>
+               <geometry>
+                    <xacro:Cube size="${slider_size}"/>
+               </geometry>
+               <material name="red"/>
+          </visual>
+     </link>
 <!-- ******************** ARM FOUR ******************* -->
      <!-- Base_link to Upper arm  -->
@@ -172,10 +205,19 @@
      </link>
      <!-- Lower Arm to rail attachment -->
-     <joint name="theta12" type="continuous">
+     <joint name="theta12" type="prismatic">
           <parent link="lowerArm_four"/>
           <child  link="railAttach_four"/>
           <origin xyz="0 0 ${bottomlimbLng}" rpy="-${pi/4} ${pi/4} 0"/>  <!-- rpy="${pi/3} ${3*pi/4} -${pi/2}"  |${pi/4} -${pi/2} 0-->
-          <axis   xyz="1 0 0"/>
-     </joint>
-     <link name="railAttach_four"/>
+          <axis   xyz="0 0 1"/>
+          <limit lower="${lLim_back}" upper="${uLim_back}" velocity="100" effort="100"/>
+     </joint>
+     <link name="railAttach_four">
+          <visual>
+               <origin xyz="-${slider_size/2} 0 0" rpy="0 0 0"/>
+               <geometry>
+                    <xacro:Cube size="${slider_size}"/>
+               </geometry>
+               <material name="red"/>
+          </visual>
+     </link>
  </robot>

File: urdf/util.xacro (robot description, xacro)
@@ -16,4 +16,9 @@
     <xacro:property name="O_y" value="${(pltf_w/2) - (limbRad + buffer) }" />
     <xacro:property name="O_z" value="${pltf_h/2}" />
+    <!-- Tempary upper and lower limits -->
+    <xacro:property name="uLim_front" value="${bottomlimbLng+toplimbLng}"/>
+    <xacro:property name="lLim_front" value="-${bottomlimbLng+toplimbLng}"/>
+    <xacro:property name="uLim_back" value="${bottomlimbLng+toplimbLng}"/>
+    <xacro:property name="lLim_back" value="-${bottomlimbLng+toplimbLng}"/>
     <xacro:macro name="Cube" params="size">
      <box size="${size} ${size} ${size}"/>

Commit message: Fix to urdf

File: urdf/tripteronBody.urdf.xacro (robot description, xacro)
@@ -5,12 +5,6 @@
 <!-- *************************************************** -->
 <xacro:include filename="util.xacro"/>
-    <link name="world"/>
-     <joint name="base_joint" type="fixed">
-        <origin xyz="1.5 1.0 0.25" rpy="0 0 0"/>
-        <parent link="world"/>
-        <child link="base_link"/>
-    </joint>
 <!-- URDF relations to IRL are in meters-->
-     <link name="base_link">
+     <link name="platform">
           <visual>
                <origin xyz="0 0 0" rpy="0 0 0"/>	<!-- Physical Center of robot Endeffector-->
@@ -24,5 +18,5 @@
      <!-- Base_link to Upper arm  -->
      <joint name="theta1" type="continuous">
-          <parent link="base_link"/>
+          <parent link="platform"/>
           <child  link="upperArm_one"/>
           <origin xyz="${O_x} -${O_y} -${O_z}" rpy="-${pi/2} -${pi/4} 0"/>
@@ -58,6 +52,6 @@
           <parent link="lowerArm_one"/>
           <child  link="railAttach_one"/>
-          <origin xyz="0 0 ${bottomlimbLng}" rpy="-${pi/4} -${pi/4} -${pi/2}"/>
-          <axis   xyz="0 1 0"/>
+          <origin xyz="0 0 ${bottomlimbLng}" rpy="0 0 0"/>
+          <axis   xyz="1 0 0"/>
      </joint>
      <link name="railAttach_one"/>
@@ -99,6 +93,6 @@
           <parent link="lowerArm_two"/>
           <child  link="railAttach_two"/>
-          <origin xyz="0 0 ${bottomlimbLng}" rpy="-${pi/4} ${pi/4} -${pi/2}"/>
-          <axis   xyz="0 1 0"/>
+          <origin xyz="0 0 ${bottomlimbLng}" rpy="0 0 0"/>
+          <axis   xyz="1 0 0"/>
      </joint>
      <link name="railAttach_two"/>
@@ -140,5 +134,5 @@
           <parent link="lowerArm_three"/>
           <child  link="railAttach_three"/>
-          <origin xyz="0 0 ${bottomlimbLng}" rpy="-${pi/4} ${pi/4} 0"/>
+          <origin xyz="0 0 ${bottomlimbLng}" rpy="0 0 0"/>
           <axis   xyz="1 0 0"/>
      </joint>
@@ -181,5 +175,5 @@
           <parent link="lowerArm_four"/>
           <child  link="railAttach_four"/>
-          <origin xyz="0 0 ${bottomlimbLng}" rpy="-${pi/4} ${pi/4} 0"/>  <!-- rpy="${pi/3} ${3*pi/4} -${pi/2}"  |${pi/4} -${pi/2} 0-->
+          <origin xyz="0 0 ${bottomlimbLng}" rpy="0 0 0"/>  <!-- rpy="${pi/3} ${3*pi/4} -${pi/2}"  |${pi/4} -${pi/2} 0-->
           <axis   xyz="1 0 0"/>
      </joint>

Commit message: basic movement

File: urdf/tripteronBody.urdf.xacro (robot description, xacro)
@@ -59,5 +59,5 @@
      <!-- Base_link to Upper arm  -->
      <joint name="theta4" type="continuous">
-          <parent link="base_link"/>
+          <parent link="platform"/>
           <child  link="upperArm_two"/>
           <origin xyz="${O_x} ${O_y} -${O_z}" rpy="-${pi/2} -${pi/4} 0"/>
@@ -100,5 +100,5 @@
      <!-- Base_link to Upper arm  -->
      <joint name="theta7" type="continuous">
-          <parent link="base_link"/>
+          <parent link="platform"/>
           <child  link="upperArm_three"/>
           <origin xyz="-${O_x} -${O_y} -${O_z}" rpy="${pi/3} ${pi/4} -${pi/4}"/>  <!-- Come back later to mess with the yaw  -${pi/4} -->
@@ -141,5 +141,5 @@
      <!-- Base_link to Upper arm  -->
      <joint name="theta10" type="continuous">
-          <parent link="base_link"/>
+          <parent link="platform"/>
           <child  link="upperArm_four"/>
           <origin xyz="-${O_x} ${O_y} -${O_z}" rpy="-${pi/3} ${pi/4} ${pi/4}"/>  <!-- Come back later to mess with the yaw  -0.7854 -->

Commit message: almost there

File: urdf/tripteronBody.urdf.xacro (robot description, xacro)
@@ -49,9 +49,8 @@
      </link>
      <!-- Lower Arm to rail attachment -->
-     <joint name="theta3" type="continuous">
+     <joint name="theta3" type="fixed">
           <parent link="lowerArm_one"/>
           <child  link="railAttach_one"/>
           <origin xyz="0 0 ${bottomlimbLng}" rpy="0 0 0"/>
-          <axis   xyz="1 0 0"/>
      </joint>
      <link name="railAttach_one"/>
@@ -90,9 +89,8 @@
      </link>
      <!-- Lower Arm to rail attachment -->
-     <joint name="theta6" type="continuous">
+     <joint name="theta6" type="fixed">
           <parent link="lowerArm_two"/>
           <child  link="railAttach_two"/>
           <origin xyz="0 0 ${bottomlimbLng}" rpy="0 0 0"/>
-          <axis   xyz="1 0 0"/>
      </joint>
      <link name="railAttach_two"/>
@@ -131,9 +129,8 @@
      </link>
      <!-- Lower Arm to rail attachment -->
-     <joint name="theta9" type="continuous">
+     <joint name="theta9" type="fixed">
           <parent link="lowerArm_three"/>
           <child  link="railAttach_three"/>
           <origin xyz="0 0 ${bottomlimbLng}" rpy="0 0 0"/>
-          <axis   xyz="1 0 0"/>
      </joint>
      <link name="railAttach_three"/>
@@ -172,9 +169,8 @@
      </link>
      <!-- Lower Arm to rail attachment -->
-     <joint name="theta12" type="continuous">
+     <joint name="theta12" type="fixed">
           <parent link="lowerArm_four"/>
           <child  link="railAttach_four"/>
           <origin xyz="0 0 ${bottomlimbLng}" rpy="0 0 0"/>  <!-- rpy="${pi/3} ${3*pi/4} -${pi/2}"  |${pi/4} -${pi/2} 0-->
-          <axis   xyz="1 0 0"/>
      </joint>
      <link name="railAttach_four"/>

File: urdf/util.xacro (robot description, xacro)
@@ -7,5 +7,5 @@
     <xacro:property name="limbRad" value="0.0127" />
     <xacro:property name="toplimbLng" value="0.1524" />
-    <xacro:property name="bottomlimbLng" value="0.2155" /> <!-- 0.2155  -->
+    <xacro:property name="bottomlimbLng" value="0.1524" /> <!-- 0.2155  -->
     <xacro:property name="pltf_l" value="0.1524" />
     <xacro:property name="pltf_w" value="0.1524" />
