Commit message: Final fixes for demo vid

File: urdf/tripteronBodyFull.urdf.xacro (robot description, xacro)
@@ -7,5 +7,5 @@
     <link name="world"/>
     <joint name="base_joint" type="fixed">
-        <origin xyz="1.5 1.0 0.25" rpy="0 0 0"/>
+        <origin xyz="0 0 0" rpy="0 0 0"/>
         <parent link="world"/>
         <child link="base_link"/>
@@ -13,11 +13,12 @@
 <!-- URDF relations to IRL are in meters-->
      <link name="base_link">
-          <visual>
-               <origin xyz="0 0 0" rpy="0 0 0"/>	<!-- Physical Center of robot Endeffector-->
-               <geometry>
-                    <box size="${pltf_l} ${pltf_w} ${pltf_h}" />
+     <link name="platform">
+     <visual>
+               <geometry>
+                    <box size="0.2 0.2 0.2" />
                </geometry>
                <material name="magenta"/>
           </visual>
+     </link>
      </link>
 <!-- ******************** ARM ONE ******************* -->
