Commit message: new urdf

File: robotDescription/tripteron.urdf.xacro (robot description, xacro)
@@ -12,5 +12,5 @@
         <parent link="base"/>
         <child  link="right_railAttach_one"/>
-        <origin xyz="0 0 0" rpy="0 0 0"/>
+        <origin xyz="0 0 ${slider_size/2}" rpy="0 0 0"/>
         <axis   xyz="1 0 0"/>
         <limit effort="1000.0" lower="0.0" upper="2.0" velocity="0.5"/>
@@ -28,12 +28,12 @@
         <parent link="right_railAttach_one"/>
         <child  link="right_lower_arm"/>
-        <origin xyz="0 0 ${slider_size}" rpy="0 ${pi/4} 0"/>
+        <origin xyz="0 0 ${slider_size/2}" rpy="0 ${pi/4} 0"/>
         <axis   xyz="1 0 0"/>
     </joint>
     <link name="right_lower_arm">
         <visual>
-            <origin xyz="0 0 -${toplimbLng/2}" rpy="0 0 0"/>
+            <origin xyz="0 0 ${bottomlimbLng/2}" rpy="0 0 0"/>
             <geometry>
-                <cylinder radius="${limbRad}" length="${toplimbLng}"/>
+                <cylinder radius="${limbRad}" length="${bottomlimbLng}"/>
             </geometry>
             <material name="cyan"/>
@@ -43,14 +43,14 @@
         <parent link="right_lower_arm"/>
         <child  link="right_upper_arm"/>
-        <origin xyz="0 0 ${slider_size}" rpy="0 -${pi/4} 0"/>
+        <origin xyz="0 0 ${bottomlimbLng}" rpy="0 0 0"/>
         <axis   xyz="1 0 0"/>
     </joint>
     <link name="right_upper_arm">
         <visual>
-            <origin xyz="0 0 -${toplimbLng/2}" rpy="0 0 0"/>
+            <origin xyz="0 0 ${toplimbLng/2}" rpy="0 0 0"/>
             <geometry>
                 <cylinder radius="${limbRad}" length="${toplimbLng}"/>
             </geometry>
-            <material name="cyan"/>
+            <material name="green"/>
         </visual>
     </link>

File: robotDescription/util.xacro (robot description, xacro)
@@ -1,11 +1,11 @@
 <?xml version="1.0"?>
 <robot xmlns:xacro="http://www.ros.org/wiki/xacro" name="tripteron">
-    <xacro:property name="limbRad" value="0.0127" />
-    <xacro:property name="toplimbLng" value="0.1524" />
-    <xacro:property name="bottomlimbLng" value="0.1524" />
-    <xacro:property name="pltf_l" value="0.1524" />
-    <xacro:property name="pltf_w" value="0.1524" />
-    <xacro:property name="pltf_h" value="0.1016" />
-    <xacro:property name="slider_size" value="0.1016" />
+    <xacro:property name="limbRad" value="0.013" />
+    <xacro:property name="toplimbLng" value="0.15" />
+    <xacro:property name="bottomlimbLng" value="0.15" />
+    <xacro:property name="pltf_l" value="0.15" />
+    <xacro:property name="pltf_w" value="0.15" />
+    <xacro:property name="pltf_h" value="0.10" />
+    <xacro:property name="slider_size" value="0.10" />
     <xacro:property name="buffer" value="0.0135" />
     <xacro:property name="O_x" value="${(pltf_l/2) - (limbRad + buffer) }" />
